Commit message: parameters

File: config/svs_tree.urdf (robot description, URDF)
Before this commit: robot StereoVisionSystem, 13 links, 12 joints
Links:
- link bl_fy: geometry visual sphere radius=0.01
- link br_fy: geometry visual sphere radius=0.01
- link fl_fy: geometry visual sphere radius=0.01
- link fr_fy: geometry visual sphere radius=0.01

Commit message: successfull unity test

File: config/svs_tree.urdf (robot description, URDF)
Before this commit: robot StereoVisionSystem, 13 links, 12 joints
Links:
- added link cam_link
Joints:
- added joint cam_to_base: type fixed, parent base_link, child cam_link, origin xyz=0 0 0 rpy=0.0 0.0 1.57
- joint base_to_bl: parent base_link -> cam_link
- joint base_to_br: parent base_link -> cam_link
- joint base_to_fl: parent base_link -> cam_link
- joint base_to_fr: parent base_link -> cam_link
- joint bl_to_l_ph: origin xyz=0 0 0 rpy=0 0.785 0 -> xyz=0 0 0 rpy=0 -0.785 0
- joint bl_to_r_ph: origin xyz=0 0 0 rpy=0 -0.785 0 -> xyz=0 0 0 rpy=0 0.785 0
- joint br_to_l_ph: origin xyz=0 0 0 rpy=0 0.785 0 -> xyz=0 0 0 rpy=0 -0.785 0
- joint br_to_r_ph: origin xyz=0 0 0 rpy=0 -0.785 0 -> xyz=0 0 0 rpy=0 0.785 0
- joint fl_to_l_ph: origin xyz=0 0 0 rpy=0 0.785 0  -> xyz=0 0 0 rpy=0 -0.785 0 
- joint fl_to_r_ph: origin xyz=0 0 0 rpy=0 -0.785 0  -> xyz=0 0 0 rpy=0 0.785 0 
- joint fr_to_l_ph: origin xyz=0 0 0 rpy=0 0.785 0 -> xyz=0 0 0 rpy=0 -0.785 0
- joint fr_to_r_ph: origin xyz=0 0 0 rpy=0 -0.785 0 -> xyz=0 0 0 rpy=0 0.785 0
